Commit message: [Sim] getting gazebo to load urdf model

File: ros-workspace/src/open_quadruped/urdf/spot_macro.xacro (robot description, xacro)
@@ -1,7 +1,4 @@
 <?xml version="1.0" ?>
 <robot xmlns:xacro="http://www.ros.org/wiki/xacro">
-  <material name="orange">
-    <color rgba="1.0 0.5 0.0 1"/>
-  </material>
   <material name="black">
     <color rgba="0.1 0.1 0.1 1"/>
@@ -51,7 +48,4 @@
         <xacro:if value="${matname == 'black'}">
           <material>Gazebo/Black</material>
-        </xacro:if>
-        <xacro:if value="${matname == 'orange'}">
-          <material>Gazebo/Orange</material>
         </xacro:if>
     </gazebo>
